File: KiCad/CanSat.kicad_pcb (KiCad board)
At the start: 4 copper layers, 50 x 55 mm, 96 parts, among them J1 GPS, J10 LED, J11 PSU_CTRL, J12 POWER, J13 SWD, J14 SDCARD, J15 DF40C-100DS-0.4V(51), J16 DF40C-100DS-0.4V(51), J17 RPI_GPIO, J2 DEPLOY, J3 TEMP, J4 ENV_SENSORS, J5 RF_DATA, J6 GND, J7 GND, J8 GND, J9 COMM_ANT, P1 USB_SDR, U1 Ai-Thinker-Ra-01, U2 DS18B20U+, U3 STM32F407VGTx, U4 SN74LVC1G125DBVR, U5 USBLC6-2SC6, U6 SN74LVC1G125DBVR, Y1 16M

Commit message: FC PCB components layout
Parts:
- removed C2, C3: 270u, Capacitor_SMD:C_Elec_8x6.2
- removed C21: 10u, Capacitor_SMD:CP_Elec_4x5.4
- removed C4, C5: 150u, Capacitor_SMD:C_Elec_6.3x5.8
- removed R15, R17, R18, R21: 22, Resistor_SMD:R_0603_1608Metric_Pad1.05x0.95mm_HandSolder
- removed R16, R20, R22, R23, R24, R25: 47k, Resistor_SMD:R_0603_1608Metric_Pad1.05x0.95mm_HandSolder
- added RN1: 47k, Resistor_SMD:R_Array_Concave_4x0603, F.Cu at (186.8, 48.1)
- added RN2: 47k, Resistor_SMD:R_Array_Concave_4x0603, F.Cu at (186.8, 43.9)
- added RN3: 22, Resistor_SMD:R_Array_Concave_4x0603, B.Cu at (197.9, 56.9)
- J9: footprint Connector_Coaxial:SMA_Wurth_60312002114503_Vertical -> Connector_Coaxial:U.FL_Molex_MCRF_73412-0110_Vertical; moved to B.Cu
- moved R33 127.9 mm to (201.1, 46.5), turned to 90 degrees
- moved J6 119.9 mm to (109.0, 51.6)
- moved J8 118.3 mm to (118.3, 51.6)
- moved J7 113.1 mm to (113.6, 51.6)
- moved J9 87.8 mm to (188.1, 75.2), turned to 270 degrees
- moved C12 1.54 mm to (197.9, 52.7)
- moved U2 0.69 mm to (188.6, 81.2)
Routing:
- net Net-(C12-Pad1): track 7.10 -> 0.00 mm
- net Net-(J13-Pad6): track 3.56 -> 0.00 mm
- net Net-(J13-Pad4): track 3.45 -> 0.00 mm
- net Net-(J13-Pad2): track 3.35 -> 0.00 mm
- net +3V3: track 15.3 -> 18.5 mm
- net /STM32 MCU/SD_CLK: track 0.00 -> 3.12 mm, vias 0 -> 1
- net /STM32 MCU/SD_DAT3: track 0.00 -> 2.40 mm, vias 0 -> 1
- net /STM32 MCU/SD_DAT1: track 0.00 -> 2.29 mm, vias 0 -> 1
- net /STM32 MCU/SD_DAT0: track 0.00 -> 2.17 mm, vias 0 -> 1
- net /STM32 MCU/SD_CMD: track 0.00 -> 2.07 mm, vias 0 -> 1
- net /STM32 MCU/SD_DAT2: track 0.00 -> 2.05 mm, vias 0 -> 1

Commit message: Semi-final flight computer version
Parts:
- removed J8: GND, Connector_PinHeader_2.54mm:PinHeader_1x02_P2.54mm_Vertical
- removed JP1: SCL, Jumper:SolderJumper-2_P1.3mm_Open_TrianglePad1.0x1.5mm
- removed JP2: SDA, Jumper:SolderJumper-2_P1.3mm_Open_TrianglePad1.0x1.5mm
- removed JP4: RPI_BOOT, TestPoint:TestPoint_2Pads_Pitch2.54mm_Drill0.8mm
- added G***: LOGO, Libs:env, F.Cu at (203.8, 83.0)
- added G***: LOGO, Libs:swd, B.Cu at (194.9, 55.9)
- added G***: LOGO, Libs:temp, F.Cu at (189.2, 63.2)
- added G***: LOGO, Libs:btn, F.Cu at (188.4, 69.6)
- added G***: LOGO, Libs:ant, F.Cu at (187.1, 75.5)
- added G***: LOGO, Libs:pwr, B.Cu at (222.8, 76.7)
- added G***: LOGO, Libs:lookmumflyingcan_cs, B.Cu at (216.7, 73.2)
- added G***: LOGO, Libs:cansat_bw, B.Cu at (216.4, 65.7)
- added G***: LOGO, Libs:chg, B.Cu at (227.8, 75.0)
- added G***: LOGO, Libs:rf, B.Cu at (225.6, 42.4)
- added G***: LOGO, Libs:gps, B.Cu at (227.0, 62.5)
- added G***: LOGO, Libs:pwr, F.Cu at (231.6, 66.9)
- added G***: LOGO, Libs:act, F.Cu at (231.6, 57.8)
- added G***: LOGO, Libs:usb, B.Cu at (210.2, 34.2)
- added G***: LOGO, Libs:usb, F.Cu at (210.2, 33.1)
- added G***: LOGO, Libs:card, B.Cu at (199.0, 34.1)
- added SCL: SCL, Jumper:SolderJumper-2_P1.3mm_Open_TrianglePad1.0x1.5mm, B.Cu at (228.1, 69.0)
- added SDA: SDA, Jumper:SolderJumper-2_P1.3mm_Open_TrianglePad1.0x1.5mm, B.Cu at (225.4, 69.0)
- added nBOOT: RPI_BOOT, TestPoint:TestPoint_2Pads_Pitch2.54mm_Drill0.8mm, B.Cu at (223.3, 48.9)
- C6, J12, R10, R11, R12, R30: moved to B.Cu
- H1, H2, H3, H4: value MountingHole -> MountingHole_Pad; footprint MountingHole:MountingHole_2.7mm_M2.5 -> MountingHole:MountingHole_2.7mm_M2.5_Pad_Via
- U4, U6: value SN74LVC1G125DBVR -> SN74LVC1G125DCKT; footprint Libs:SOT95P280X145-5N -> Libs:SOT65P210X110-5N
- moved J6 82.8 mm to (189.5, 32.4)
- moved J7 75.9 mm to (187.1, 32.4)
- moved C16 34.0 mm to (214.4, 39.5), turned to 180 degrees
- moved U4 33.3 mm to (231.8, 34.5)
- moved C11 31.1 mm to (202.6, 42.9), turned to 90 degrees
- moved U6 26.8 mm to (224.2, 40.7)
- moved R33 21.2 mm to (221.6, 41.0), turned to 270 degrees
- moved R9 20.4 mm to (205.6, 70.6), turned to 270 degrees
- moved R30 15.6 mm to (224.3, 46.8)
- moved J17 15.1 mm to (222.8, 69.4)
- moved C9 14.3 mm to (207.8, 60.1)
- moved C15 12.6 mm to (216.9, 59.3), turned to 180 degrees
- moved C18 11.1 mm to (220.3, 60.9), turned to 0 degrees
- moved C17 11.1 mm to (220.4, 62.5), turned to 0 degrees
- moved L1 10.5 mm to (218.8, 64.0), turned to 0 degrees
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Connections:
- H1 pad 1: (no net) -> GND
- H2 pad 1: (no net) -> GND
- H3 pad 1: (no net) -> GND
- H4 pad 1: (no net) -> GND
- J15 pad 99: /RPi CM4/GLOBAL_EN -> /RPi CM4/RPI_ENABLE
- R13 pad 2: /Peripherals and Connectors/SCL -> /Peripherals and Connectors/SDA
- R14 pad 2: /Peripherals and Connectors/SDA -> /Peripherals and Connectors/SCL
- U3 pad 1: /Power/PWR_CRITICAL -> /Peripherals and Connectors/GPIO_2
- U3 pad 15: /STM32 MCU/LED1 -> Net-(U3-Pad15)
- U3 pad 16: /STM32 MCU/LED2 -> Net-(U3-Pad16)
- U3 pad 17: Net-(U3-Pad17) -> /Peripherals and Connectors/LED_DATA
- U3 pad 2: /Power/PWR_WARN -> Net-(U3-Pad2)
- U3 pad 3: /Power/PWR_VALID -> /Peripherals and Connectors/GPIO_3
- U3 pad 35: /Peripherals and Connectors/LED_DATA -> Net-(U3-Pad35)
- U3 pad 36: /Peripherals and Connectors/DEPLOY -> Net-(U3-Pad36)
- U3 pad 37: /Peripherals and Connectors/DS_EXTERNAL -> Net-(U3-Pad37)
- U3 pad 38: Net-(U3-Pad38) -> /Power/PWR_VALID
- U3 pad 39: Net-(U3-Pad39) -> /Power/PWR_WARN
- U3 pad 4: Net-(U3-Pad4) -> /RPi CM4/GLOBAL_EN
- U3 pad 40: Net-(U3-Pad40) -> /Power/PWR_CRITICAL
- U3 pad 42: /Peripherals and Connectors/GPIO_2 -> Net-(U3-Pad42)
- U3 pad 43: Net-(U3-Pad43) -> /Peripherals and Connectors/DEPLOY
- U3 pad 44: Net-(U3-Pad44) -> /Peripherals and Connectors/DS_EXTERNAL
- U3 pad 46: /Peripherals and Connectors/GPIO_3 -> Net-(U3-Pad46)
- U3 pad 5: Net-(U3-Pad5) -> /RPi CM4/RUN_PG
- U3 pad 70: /RPi CM4/RUN_PG -> Net-(U3-Pad70)
- U3 pad 71: /RPi CM4/GLOBAL_EN -> Net-(U3-Pad71)
- U3 pad 91: Net-(U3-Pad91) -> /STM32 MCU/LED1
- U3 pad 93: /Peripherals and Connectors/SDA -> /STM32 MCU/LED2
- U3 pad 96: Net-(U3-Pad96) -> /Peripherals and Connectors/SDA
- U6 pad 4: /RPi CM4/GLOBAL_EN -> /RPi CM4/RPI_ENABLE
Routing:
- net +3V3: track 18.5 -> 277.6 mm, vias 0 -> 36
- net +5V: track 8.49 -> 120.7 mm, vias 0 -> 7
- net GND: track 6.18 -> 117.5 mm, vias 0 -> 98
- net /Peripherals and Connectors/SDA: track 7.18 -> 95.6 mm, vias 0 -> 3
- net /Peripherals and Connectors/SCL: track 12.4 -> 91.2 mm, vias 2 -> 6
- net /Peripherals and Connectors/DS_EXTERNAL: track 0.00 -> 68.1 mm, vias 0 -> 5
- net VBAT: track 0.00 -> 57.1 mm, vias 0 -> 1
- net /RPi CM4/USB-: track 0.00 -> 34.0 mm, vias 0 -> 1
- net Net-(R32-Pad2): track 2.23 -> 34.9 mm, vias 0 -> 2
- net /Peripherals and Connectors/RADIO_RST: track 0.00 -> 31.8 mm, vias 0 -> 4
- net /RPi CM4/USB+: track 0.00 -> 31.5 mm, vias 0 -> 1
- net /Power/PWR_CRITICAL: track 0.00 -> 30.1 mm, vias 0 -> 2
- net /Power/PWR_WARN: track 0.00 -> 29.2 mm, vias 0 -> 2
- net /RPi CM4/RPI_TX: track 0.00 -> 29.1 mm, vias 0 -> 3
- net /RPi CM4/RPI_RX: track 0.00 -> 28.9 mm, vias 0 -> 3
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- added copper zone on B.Cu, net GND
- added copper zone on F.Cu, net GND
- added copper zone on In1.Cu, net GND
Other:
- net class Default: clearance 0.2 -> 0.0889; via_dia 0.8 -> 0.45; via_drill 0.4 -> 0.2
- rule trace_clearance: 0.2 -> 0.0889
- rule via_min_drill: 0.3 -> 0.2
- rule via_min_size: 0.4 -> 0.45
- board text added: "v.1"
