File: KiCad/mcu.sch (KiCad schematic (older format))
At the start: 22 parts

Commit message: Update schematic
Connections:
- net labels added: GLOBAL_EN, RUN_PG
Changed lines of the file:
@@
 encoding utf-8
 Sheet 5 5
-Title ""
+Title "STM32F4 MCU Section"
 Date "2020-12-03"
 Rev "V0.1"
@@
 Text HLabel 3450 3650 2    50   BiDi ~ 0
 DS_TEMP
+Text HLabel 3450 2850 2    50   BiDi ~ 0
+RUN_PG
+Text HLabel 3450 2950 2    50   Output ~ 0
+GLOBAL_EN
 $EndSCHEMATC

Commit message: Finalized schematic and created S/F associations
Parts:
- removed R?: 4k7, symbol Device:R_Small
- removed Y?: 16M, symbol Device:Crystal
- added C12: 1u, Capacitor_SMD:C_0603_1608Metric_Pad1.05x0.95mm_HandSolder, symbol Device:C_Small
- added C21: 10u, Capacitor_SMD:CP_Elec_4x5.4, symbol Device:CP_Small
- added C22, C9: 100n, Capacitor_SMD:C_0603_1608Metric_Pad1.05x0.95mm_HandSolder, symbol Device:C_Small
- added D3: LED1, LED_SMD:LED_0603_1608Metric_Pad1.05x0.95mm_HandSolder, symbol Device:LED
- added D4: LED2, LED_SMD:LED_0603_1608Metric_Pad1.05x0.95mm_HandSolder, symbol Device:LED
- added J13: SWD, Connector_PinHeader_1.27mm:PinHeader_2x05_P1.27mm_Vertical_SMD, symbol Connector_Generic:Conn_02x05_Odd_Even
- added R13: 4k7, Resistor_SMD:R_0603_1608Metric_Pad1.05x0.95mm_HandSolder, symbol Device:R_Small
- added R15, R17, R18, R21: 22, Resistor_SMD:R_0603_1608Metric_Pad1.05x0.95mm_HandSolder, symbol Device:R_Small
- added R16, R20, R22, R23, R24, R25: 47k, Resistor_SMD:R_0603_1608Metric_Pad1.05x0.95mm_HandSolder, symbol Device:R_Small
- added R26: 10k, Resistor_SMD:R_0603_1608Metric_Pad1.05x0.95mm_HandSolder, symbol Device:R_Small
- added R28, R29: 470, Resistor_SMD:R_0603_1608Metric_Pad1.05x0.95mm_HandSolder, symbol Device:R
- added Y1: 16M, Crystal:Crystal_SMD_3225-4Pin_3.2x2.5mm_HandSoldering, symbol Device:Crystal_GND24_Small
- C10, C11, C13, C14, C15, C16, C17, C18, C19, C20, C6, C7, C8: renamed from C?; footprint (none) -> Capacitor_SMD:C_0603_1608Metric_Pad1.05x0.95mm_HandSolder
- J14: renamed from J?; footprint MOLEX_47352-1001 -> Libs:MOLEX_47352-1001
- JP3: renamed from JP?; value BOOT -> STM_BOOT; footprint (none) -> Jumper:SolderJumper-3_P1.3mm_Bridged12_RoundedPad1.0x1.5mm
- L1: renamed from L?; footprint (none) -> Inductor_SMD:L_0603_1608Metric_Pad1.05x0.95mm_HandSolder
- R14: renamed from R?; footprint (none) -> Resistor_SMD:R_0603_1608Metric_Pad1.05x0.95mm_HandSolder
- R19: renamed from R?; value 47R -> 47; footprint (none) -> Resistor_SMD:R_0603_1608Metric_Pad1.05x0.95mm_HandSolder
- R27: renamed from R?; footprint (none) -> Resistor_SMD:R_0805_2012Metric_Pad1.15x1.40mm_HandSolder
- gave numbers to parts that had none: 1
Connections:
- net labels added: GPIO_2, GPIO_3, LED1, LED2, NRST, PWR_CRITICAL, PWR_VALID, PWR_WARN, SWCLK, SWDIO, SWO
- wire segments 91 -> 151
- no-connect marks 0 -> 51
Other:
- note added: "place near SD card"
- moved on the sheet: C11, C14, C15, C16, C17, C18, C19, C20, C8, J14, JP3, L1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

Commit message: Done some stuff
Parts:
- removed C21: 10u, Capacitor_SMD:CP_Elec_4x5.4, symbol Device:CP_Small
- removed R16, R20, R22, R23, R24, R25: 47k, Resistor_SMD:R_0603_1608Metric_Pad1.05x0.95mm_HandSolder, symbol Device:R_Small
- added RN1: 47k, Resistor_THT:R_Array_SIP7, symbol Device:R_Network06
Connections:
- net +3V3: now also RN1.1 (common)
- net SD_CLK: now also RN1.2 (R1)
- net SD_CMD: now also RN1.3 (R2)
- net SD_DAT0: now also RN1.7 (R6)
- net SD_DAT1: now also RN1.6 (R5)
- net SD_DAT2: now also RN1.5 (R4)
- net SD_DAT3: now also RN1.4 (R3)
Other:
- moved on the sheet: C22
Changed lines of the file:
@@
 Text Label 7200 3900 0    50   ~ 0
 SD_DAT2
-Text Label 3800 5950 2    50   ~ 0
-SD_DAT0
 Wire Wire Line
 	3450 5950 3800 5950
@@
 NoConn ~ 2250 1450
 Wire Wire Line
-	7400 4500 7400 4400
-Wire Wire Line
-	7400 4400 7500 4400
-$Comp
-L Device:R_Small R25
-U 1 1 5FCF20B5
-P 7050 4350
-F 0 "R25" H 7109 4396 50  0000 L CNN
-F 1 "47k" H 7109 4305 50  0000 L CNN
-F 2 "Resistor_SMD:R_0603_1608Metric_Pad1.05x0.95mm_HandSolder" H 7050 4350 50  0001 C CNN
-F 3 "~" H 7050 4350 50  0001 C CNN
-	1    7050 4350
-	1    0    0    -1
-$EndComp
-Wire Wire Line
-	7050 4450 7050 4500
-Connection ~ 7050 4500
-Wire Wire Line
-	7050 4500 7400 4500
-$Comp
-L Device:R_Small R24
-U 1 1 5FCF6430
-P 6800 4350
-F 0 "R24" H 6859 4396 50  0000 L CNN
-F 1 "47k" H 6859 4305 50  0000 L CNN
-F 2 "Resistor_SMD:R_0603_1608Metric_Pad1.05x0.95mm_HandSolder" H 6800 4350 50  0001 C CNN
-F 3 "~" H 6800 4350 50  0001 C CNN
-	1    6800 4350
-	1    0    0    -1
-$EndComp
-Wire Wire Line
-	6800 4450 6800 4500
-$Comp
-L Device:R_Small R23
-U 1 1 5FCF8F30
-P 6550 4350
-F 0 "R23" H 6609 4396 50  0000 L CNN
-F 1 "47k" H 6609 4305 50  0000 L CNN
-F 2 "Resistor_SMD:R_0603_1608Metric_Pad1.05x0.95mm_HandSolder" H 6550 4350 50  0001 C CNN
-F 3 "~" H 6550 4350 50  0001 C CNN
-	1    6550 4350
-	1    0    0    -1
-$EndComp
-Wire Wire Line
-	6550 4450 6550 4500
-$Comp
-L Device:R_Small R22
-U 1 1 5FCFBB74
-P 6300 4350
-F 0 "R22" H 6359 4396 50  0000 L CNN
-F 1 "47k" H 6359 4305 50  0000 L CNN
-F 2 "Resistor_SMD:R_0603_1608Metric_Pad1.05x0.95mm_HandSolder" H 6300 4350 50  0001 C CNN
-F 3 "~" H 6300 4350 50  0001 C CNN
-	1    6300 4350
-	1    0    0    -1
-$EndComp
-Wire Wire Line
-	6300 4450 6300 4500
-Connection ~ 6800 4500
-Wire Wire Line
-	6800 4500 7050 4500
-Connection ~ 6550 4500
-Wire Wire Line
-	6550 4500 6800 4500
-$Comp
-L Device:R_Small R20
-U 1 1 5FCFF123
-P 6050 4350
-F 0 "R20" H 6109 4396 50  0000 L CNN
-F 1 "47k" H 6109 4305 50  0000 L CNN
-F 2 "Resistor_SMD:R_0603_1608Metric_Pad1.05x0.95mm_HandSolder" H 6050 4350 50  0001 C CNN
-F 3 "~" H 6050 4350 50  0001 C CNN
-	1    6050 4350
-	1    0    0    -1
-$EndComp
-Wire Wire Line
-	6050 4450 6050 4500
-$Comp
-L Device:R_Small R16
-U 1 1 5FD01F7B
-P 5800 4350
-F 0 "R16" H 5859 4396 50  0000 L CNN
-F 1 "47k" H 5859 4305 50  0000 L CNN
-F 2 "Resistor_SMD:R_0603_1608Metric_Pad1.05x0.95mm_HandSolder" H 5800 4350 50  0001 C CNN
-F 3 "~" H 5800 4350 50  0001 C CNN
-	1    5800 4350
-	1    0    0    -1
-$EndComp
-Wire Wire Line
-	5800 4450 5800 4500
-Wire Wire Line
-	5800 4500 6050 4500
-Connection ~ 6050 4500
-Wire Wire Line
-	6050 4500 6300 4500
-Connection ~ 6300 4500
-Wire Wire Line
-	6300 4500 6550 4500
-Wire Wire Line
-	7050 4200 7050 4250
-Wire Wire Line
 	7050 4200 7500 4200
-Wire Wire Line
-	6800 4100 6800 4250
-Wire Wire Line
-	6800 4100 7500 4100
-Wire Wire Line
-	6550 4000 6550 4250
-Wire Wire Line
-	6550 4000 7500 4000
-Wire Wire Line
-	6300 3900 6300 4250
-Wire Wire Line
-	6300 3900 7500 3900
-Wire Wire Line
-	6050 3800 6050 4250
-Wire Wire Line
-	6050 3800 7500 3800
-Wire Wire Line
-	5800 3700 5800 4250
-Wire Wire Line
-	5800 3700 7500 3700
 $Comp
 L Device:C_Small C22
 U 1 1 5FD49E73
-P 9250 4100
-F 0 "C22" H 9342 4146 50  0000 L CNN
-F 1 "100n" H 9342 4055 50  0000 L CNN
-F 2 "Capacitor_SMD:C_0603_1608Metric_Pad1.05x0.95mm_HandSolder" H 9250 4100 50  0001 C CNN
-F 3 "~" H 9250 4100 50  0001 C CNN
-	1    9250 4100
-	1    0    0    -1
-$EndComp
-$Comp
-L Device:CP_Small C21
-U 1 1 5FD49E79
 P 8900 4100
-F 0 "C21" H 8988 4146 50  0000 L CNN
-F 1 "10u" H 8988 4055 50  0000 L CNN
-F 2 "Capacitor_SMD:CP_Elec_4x5.4" H 8900 4100 50  0001 C CNN
+F 0 "C22" H 8992 4146 50  0000 L CNN
+F 1 "100n" H 8992 4055 50  0000 L CNN
+F 2 "Capacitor_SMD:C_0603_1608Metric_Pad1.05x0.95mm_HandSolder" H 8900 4100 50  0001 C CNN
 F 3 "~" H 8900 4100 50  0001 C CNN
 	1    8900 4100
 	1    0    0    -1
 $EndComp
-Wire Wire Line
-	8900 4000 9250 4000
 $Comp
 L power:GND #PWR0139
@@
 Wire Wire Line
 	8900 4200 8900 4250
-Wire Wire Line
-	8900 4200 9250 4200
-Connection ~ 8900 4200
 $Comp
 L power:+3V3 #PWR0140
 U 1 1 5FD77515
-P 5600 4500
-F 0 "#PWR0140" H 5600 4350 50  0001 C CNN
-F 1 "+3V3" H 5615 4673 50  0000 C CNN
-F 2 "" H 5600 4500 50  0001 C CNN
-F 3 "" H 5600 4500 50  0001 C CNN
-	1    5600 4500
-	1    0    0    -1
-$EndComp
-Wire Wire Line
-	5600 4500 5800 4500
-Connection ~ 5800 4500
+P 6350 4550
+F 0 "#PWR0140" H 6350 4400 50  0001 C CNN
+F 1 "+3V3" H 6365 4723 50  0000 C CNN
+F 2 "" H 6350 4550 50  0001 C CNN
+F 3 "" H 6350 4550 50  0001 C CNN
+	1    6350 4550
+	1    0    0    -1
+$EndComp
 $Comp
 L power:+3V3 #PWR0141
@@
 Text Notes 8800 4550 0    50   ~ 0
 place near SD card
-Connection ~ 8900 4000
 Text HLabel 1650 4550 0    50   BiDi ~ 0
 GPIO_2
@@
 	5650 2550 5650 2600
 Connection ~ 5650 2600
+Text Label 3800 5950 2    50   ~ 0
+SD_DAT0
+$Comp
+L Device:R_Network06 RN1
+U 1 1 5FDD3900
+P 6750 4400
+F 0 "RN1" H 6370 4354 50  0000 R CNN
+F 1 "47k" H 6370 4445 50  0000 R CNN
+F 2 "Resistor_THT:R_Array_SIP7" V 7125 4400 50  0001 C CNN
+F 3 "http://www.vishay.com/docs/31509/csc.pdf" H 6750 4400 50  0001 C CNN
+	1    6750 4400
+	-1   0    0    1
+$EndComp
+Wire Wire Line
+	7500 4100 6950 4100
+Wire Wire Line
+	6950 4100 6950 4200
+Wire Wire Line
+	7500 4000 6850 4000
+Wire Wire Line
+	6850 4000 6850 4200
+Wire Wire Line
+	7500 3900 6750 3900
+Wire Wire Line
+	6750 3900 6750 4200
+Wire Wire Line
+	7500 3800 6650 3800
+Wire Wire Line
+	6650 3800 6650 4200
+Wire Wire Line
+	7500 3700 6550 3700
+Wire Wire Line
+	6550 3700 6550 4200
+Wire Wire Line
+	6350 4550 6350 4650
+Wire Wire Line
+	6350 4650 7050 4650
+Wire Wire Line
+	7050 4650 7050 4600
+Wire Wire Line
+	7500 4400 7350 4400
+Wire Wire Line
+	7350 4400 7350 4650
+Wire Wire Line
+	7350 4650 7050 4650
+Connection ~ 7050 4650
 $EndSCHEMATC

Commit message: FC PCB components layout
Parts:
- removed R15, R17, R18, R21: 22, Resistor_SMD:R_0603_1608Metric_Pad1.05x0.95mm_HandSolder, symbol Device:R_Small
- removed RN1: 47k, Resistor_THT:R_Array_SIP7, symbol Device:R_Network06
- added RN1, RN2: 47k, Resistor_SMD:R_Array_Concave_4x0603, symbol Device:R_Pack04
- added RN3: 22, Resistor_SMD:R_Array_Concave_4x0603, symbol Device:R_Pack04
Connections:
- net +3V3: now also RN1.7 (R2.2), RN1.8 (R1.2), RN2.1 (R1.1), RN2.2 (R2.1), RN2.3 (R3.1), RN2.4 (R4.1)
- net NRST: now also RN3.1 (R1.1)
- net SD_CLK: now also RN2.5 (R4.2)
- net SD_CMD: now also RN2.6 (R3.2)
- net SD_DAT0: now also RN1.2 (R2.1)
- net SD_DAT1: now also RN1.1 (R1.1)
- net SD_DAT2: now also RN2.8 (R1.2)
- net SD_DAT3: now also RN2.7 (R2.2)
- net SWCLK: now also RN3.3 (R3.1)
- net SWDIO: now also RN3.4 (R4.1)
- net SWO: now also RN3.2 (R2.1)
- net at C12.1, J13.10 (Pin_10): now also RN3.8 (R1.2)
- net at J13.2 (Pin_2): now also RN3.5 (R4.2)
- net at J13.4 (Pin_4): now also RN3.6 (R3.2)
- net at J13.6 (Pin_6): now also RN3.7 (R2.2)
- no-connect marks 51 -> 55
Changed lines of the file:
@@
 L power:+3V3 #PWR0140
 U 1 1 5FD77515
-P 6350 4550
-F 0 "#PWR0140" H 6350 4400 50  0001 C CNN
-F 1 "+3V3" H 6365 4723 50  0000 C CNN
-F 2 "" H 6350 4550 50  0001 C CNN
-F 3 "" H 6350 4550 50  0001 C CNN
-	1    6350 4550
+P 5750 4600
+F 0 "#PWR0140" H 5750 4450 50  0001 C CNN
+F 1 "+3V3" H 5765 4773 50  0000 C CNN
+F 2 "" H 5750 4600 50  0001 C CNN
+F 3 "" H 5750 4600 50  0001 C CNN
+	1    5750 4600
 	1    0    0    -1
 $EndComp
@@
 Text Label 6500 5450 2    50   ~ 0
 SWDIO
-$Comp
-L Device:R_Small R15
-U 1 1 5FFB97F1
-P 5750 5450
-F 0 "R15" V 5554 5450 50  0000 C CNN
-F 1 "22" V 5645 5450 50  0000 C CNN
-F 2 "Resistor_SMD:R_0603_1608Metric_Pad1.05x0.95mm_HandSolder" H 5750 5450 50  0001 C CNN
-F 3 "~" H 5750 5450 50  0001 C CNN
-	1    5750 5450
-	0    1    1    0
-$EndComp
-Wire Wire Line
-	5850 5450 6500 5450
+Wire Wire Line
+	6250 5450 6500 5450
 Text Label 6500 5550 2    50   ~ 0
 SWCLK
-$Comp
-L Device:R_Small R17
-U 1 1 5FFD99D3
-P 5950 5550
-F 0 "R17" V 5754 5550 50  0000 C CNN
-F 1 "22" V 5845 5550 50  0000 C CNN
-F 2 "Resistor_SMD:R_0603_1608Metric_Pad1.05x0.95mm_HandSolder" H 5950 5550 50  0001 C CNN
-F 3 "~" H 5950 5550 50  0001 C CNN
-	1    5950 5550
-	0    1    1    0
-$EndComp
-Wire Wire Line
-	6050 5550 6500 5550
+Wire Wire Line
+	6250 5550 6500 5550
 Text Label 6500 5650 2    50   ~ 0
 SWO
-$Comp
-L Device:R_Small R21
-U 1 1 5FFDECCF
-P 6150 5650
-F 0 "R21" V 5954 5650 50  0000 C CNN
-F 1 "22" V 6045 5650 50  0000 C CNN
-F 2 "Resistor_SMD:R_0603_1608Metric_Pad1.05x0.95mm_HandSolder" H 6150 5650 50  0001 C CNN
-F 3 "~" H 6150 5650 50  0001 C CNN
-	1    6150 5650
-	0    1    1    0
-$EndComp
 Wire Wire Line
 	6250 5650 6500 5650
-Wire Wire Line
-	5650 5550 5850 5550
-Wire Wire Line
-	5650 5650 6050 5650
 NoConn ~ 5650 5750
 Text Label 1400 1750 0    50   ~ 0
@@
 Wire Wire Line
 	1400 1750 1650 1750
-Text Label 6300 5850 2    50   ~ 0
+Text Label 6500 5750 2    50   ~ 0
 NRST
 $Comp
@@
 	1    0    0    -1
 $EndComp
-$Comp
-L Device:R_Small R18
-U 1 1 60044A42
-P 5950 5850
-F 0 "R18" V 5754 5850 50  0000 C CNN
-F 1 "22" V 5845 5850 50  0000 C CNN
-F 2 "Resistor_SMD:R_0603_1608Metric_Pad1.05x0.95mm_HandSolder" H 5950 5850 50  0001 C CNN
-F 3 "~" H 5950 5850 50  0001 C CNN
-	1    5950 5850
-	0    1    1    0
-$EndComp
 Wire Wire Line
 	5650 5850 5750 5850
@@
 Connection ~ 5750 5850
 Wire Wire Line
-	5750 5850 5850 5850
-Wire Wire Line
-	6050 5850 6300 5850
+	6250 5750 6500 5750
 $Comp
 L Device:Crystal_GND24_Small Y1
@@
 Text Label 3800 5950 2    50   ~ 0
 SD_DAT0
-$Comp
-L Device:R_Network06 RN1
-U 1 1 5FDD3900
-P 6750 4400
-F 0 "RN1" H 6370 4354 50  0000 R CNN
-F 1 "47k" H 6370 4445 50  0000 R CNN
-F 2 "Resistor_THT:R_Array_SIP7" V 7125 4400 50  0001 C CNN
-F 3 "http://www.vishay.com/docs/31509/csc.pdf" H 6750 4400 50  0001 C CNN
-	1    6750 4400
-	-1   0    0    1
-$EndComp
 Wire Wire Line
 	7500 4100 6950 4100
@@
 	6550 3700 6550 4200
 Wire Wire Line
-	6350 4550 6350 4650
-Wire Wire Line
-	6350 4650 7050 4650
+	5750 4600 5750 4650
 Wire Wire Line
 	7050 4650 7050 4600
@@
 	7350 4650 7050 4650
 Connection ~ 7050 4650
+$Comp
+L Device:R_Pack04 RN2
+U 1 1 5FE32852
+P 6950 4400
+F 0 "RN2" H 7138 4446 50  0000 L CNN
+F 1 "47k" H 7138 4355 50  0000 L CNN
+F 2 "Resistor_SMD:R_Array_Concave_4x0603" V 7225 4400 50  0001 C CNN
+F 3 "~" H 6950 4400 50  0001 C CNN
+	1    6950 4400
+	1    0    0    -1
+$EndComp
+Wire Wire Line
+	6950 4600 6950 4650
+Connection ~ 6950 4650
+Wire Wire Line
+	6950 4650 7050 4650
+Wire Wire Line
+	6850 4600 6850 4650
+Connection ~ 6850 4650
+Wire Wire Line
+	6850 4650 6950 4650
+Wire Wire Line
+	6750 4600 6750 4650
+Connection ~ 6750 4650
+Wire Wire Line
+	6750 4650 6850 4650
+Wire Wire Line
+	6650 4600 6650 4650
+Connection ~ 6650 4650
+Wire Wire Line
+	6650 4650 6750 4650
+Wire Wire Line
+	6550 4600 6550 4650
+Connection ~ 6550 4650
+Wire Wire Line
+	6550 4650 6650 4650
+$Comp
+L Device:R_Pack04 RN1
+U 1 1 5FE7310C
+P 6450 4400
+F 0 "RN1" H 6800 4350 50  0000 R CNN
+F 1 "47k" H 6800 4450 50  0000 R CNN
+F 2 "Resistor_SMD:R_Array_Concave_4x0603" V 6725 4400 50  0001 C CNN
+F 3 "~" H 6450 4400 50  0001 C CNN
+	1    6450 4400
+	-1   0    0    1
+$EndComp
+Wire Wire Line
+	5750 4650 6550 4650
+NoConn ~ 6350 4200
+NoConn ~ 6450 4200
+NoConn ~ 6350 4600
+NoConn ~ 6450 4600
+$Comp
+L Device:R_Pack04 RN3
+U 1 1 5FEA5572
+P 6050 5550
+F 0 "RN3" V 6375 5550 50  0000 C CNN
+F 1 "22" V 6284 5550 50  0000 C CNN
+F 2 "Resistor_SMD:R_Array_Concave_4x0603" V 6325 5550 50  0001 C CNN
+F 3 "~" H 6050 5550 50  0001 C CNN
+	1    6050 5550
+	0    -1   -1   0
+$EndComp
+Wire Wire Line
+	5650 5450 5850 5450
+Wire Wire Line
+	5650 5550 5850 5550
+Wire Wire Line
+	5850 5650 5650 5650
+Wire Wire Line
+	5750 5850 5750 5750
+Wire Wire Line
+	5750 5750 5850 5750
 $EndSCHEMATC

Commit message: Semi-final flight computer version
Connections:
- net DEPLOY: now also U3.43 (PE12); no longer U3.36 (PB1)
- net DS_TEMP: now also U3.44 (PE13); no longer U3.37 (PB2)
- net GLOBAL_EN: now also U3.4 (PE5); no longer U3.71 (PA12)
- net GPIO_2: now also U3.1 (PE2); no longer U3.42 (PE11)
- net GPIO_3: now also U3.3 (PE4); no longer U3.46 (PE15)
- net LED1: now also U3.91 (PB5); no longer U3.15 (PC0)
- net LED2: now also U3.93 (PB7); no longer U3.16 (PC1)
- net LED_DATA: now also U3.17 (PC2); no longer U3.35 (PB0)
- net PWR_CRITICAL: now also U3.40 (PE9); no longer U3.1 (PE2)
- net PWR_VALID: now also U3.38 (PE7); no longer U3.3 (PE4)
- net PWR_WARN: now also U3.39 (PE8); no longer U3.2 (PE3)
- net RUN_PG: now also U3.5 (PE6); no longer U3.70 (PA11)
- net SCL: now also R14.2; no longer R13.2
- net SDA: now also R13.2, U3.96 (PB9); no longer R14.2, U3.93 (PB7)
Other:
- moved on the sheet: R13, R14
Changed lines of the file:
@@
 $EndDescr
-$Comp
-L MCU_ST_STM32F4:STM32F407VGTx U3
-U 1 1 5FCFB0B5
-P 2550 4150
-F 0 "U3" H 2900 1500 50  0000 C CNN
-F 1 "STM32F407VGTx" H 3150 1400 50  0000 C CNN
-F 2 "Package_QFP:LQFP-100_14x14mm_P0.5mm" H 1850 1550 50  0001 R CNN
-F 3 "http://www.st.com/st-web-ui/static/active/en/resource/technical/document/datasheet/DM00037051.pdf" H 2550 4150 50  0001 C CNN
-	1    2550 4150
-	1    0    0    -1
-$EndComp
 $Comp
 L MOLEX_SD_473521001:47352-1001 J14
@@
 Text Label 2350 1200 3    50   ~ 0
 VDD
-Wire Wire Line
-	2350 1200 2350 1400
 Text Label 2950 1200 3    50   ~ 0
 VDDA
@@
 L Device:R_Small R14
 U 1 1 5FE292F5
-P 4000 4000
-F 0 "R14" H 4059 4046 50  0000 L CNN
-F 1 "4k7" H 4059 3955 50  0000 L CNN
-F 2 "Resistor_SMD:R_0603_1608Metric_Pad1.05x0.95mm_HandSolder" H 4000 4000 50  0001 C CNN
-F 3 "~" H 4000 4000 50  0001 C CNN
-	1    4000 4000
-	1    0    0    -1
-$EndComp
-Wire Wire Line
-	4000 3900 3750 3900
-Wire Wire Line
-	4000 3850 4000 3900
-Connection ~ 4000 3900
+P 4150 4100
+F 0 "R14" H 4209 4146 50  0000 L CNN
+F 1 "4k7" H 4209 4055 50  0000 L CNN
+F 2 "Resistor_SMD:R_0603_1608Metric_Pad1.05x0.95mm_HandSolder" H 4150 4100 50  0001 C CNN
+F 3 "~" H 4150 4100 50  0001 C CNN
+	1    4150 4100
+	1    0    0    -1
+$EndComp
+Wire Wire Line
+	4150 4000 3900 4000
+Wire Wire Line
+	4150 3950 4150 4000
 $Comp
 L power:+3V3 #PWR0134
 U 1 1 5FE2EDA2
-P 4000 3850
-F 0 "#PWR0134" H 4000 3700 50  0001 C CNN
-F 1 "+3V3" H 4015 4023 50  0000 C CNN
-F 2 "" H 4000 3850 50  0001 C CNN
-F 3 "" H 4000 3850 50  0001 C CNN
-	1    4000 3850
-	1    0    0    -1
-$EndComp
-Text HLabel 4200 4150 2    50   BiDi ~ 0
+P 4150 3950
+F 0 "#PWR0134" H 4150 3800 50  0001 C CNN
+F 1 "+3V3" H 4165 4123 50  0000 C CNN
+F 2 "" H 4150 3950 50  0001 C CNN
+F 3 "" H 4150 3950 50  0001 C CNN
+	1    4150 3950
+	1    0    0    -1
+$EndComp
+Text HLabel 4350 4350 2    50   BiDi ~ 0
 SDA
-Text HLabel 4200 4250 2    50   Output ~ 0
+Text HLabel 4350 4250 2    50   Output ~ 0
 SCL
 Text HLabel 3450 2150 2    50   Output ~ 0
@@
 	1    0    0    -1
 $EndComp
-Text HLabel 3450 3450 2    50   Output ~ 0
+Text HLabel 3450 5350 2    50   Output ~ 0
 LED_DATA
-Text HLabel 3450 3550 2    50   Input ~ 0
+Text HLabel 1650 4650 0    50   Input ~ 0
 DEPLOY
-Text HLabel 3450 3650 2    50   BiDi ~ 0
+Text HLabel 1650 4750 0    50   BiDi ~ 0
 DS_TEMP
-Text HLabel 3450 2850 2    50   BiDi ~ 0
+Text HLabel 1650 4050 0    50   BiDi ~ 0
 RUN_PG
-Text HLabel 3450 2950 2    50   Output ~ 0
+Text HLabel 1650 3950 0    50   Output ~ 0
 GLOBAL_EN
-Text HLabel 1650 3650 0    50   Input ~ 0
-PWR_CRITICAL
-Text HLabel 1650 3750 0    50   Input ~ 0
-PWR_WARN
-Text HLabel 1650 3850 0    50   Input ~ 0
-PWR_VALID
 NoConn ~ 7500 4300
 NoConn ~ 2250 1450
@@
 Text Notes 8800 4550 0    50   ~ 0
 place near SD card
-Text HLabel 1650 4550 0    50   BiDi ~ 0
+Text HLabel 1650 3650 0    50   BiDi ~ 0
 GPIO_2
-Text HLabel 1650 4950 0    50   BiDi ~ 0
+Text HLabel 1650 3850 0    50   BiDi ~ 0
 GPIO_3
 Wire Wire Line
-	4000 4100 4000 4150
-Connection ~ 4000 4150
-Wire Wire Line
-	4000 4150 4200 4150
+	4150 4200 4150 4250
+Connection ~ 4150 4250
+Wire Wire Line
+	4150 4250 4350 4250
 $Comp
 L Device:R_Small R13
 U 1 1 5FE2024B
-P 3750 4000
-F 0 "R13" H 3809 4046 50  0000 L CNN
-F 1 "4k7" H 3809 3955 50  0000 L CNN
-F 2 "Resistor_SMD:R_0603_1608Metric_Pad1.05x0.95mm_HandSolder" H 3750 4000 50  0001 C CNN
-F 3 "~" H 3750 4000 50  0001 C CNN
-	1    3750 4000
-	1    0    0    -1
-$EndComp
-Wire Wire Line
-	3750 4100 3750 4250
-Connection ~ 3750 4250
-Wire Wire Line
-	3750 4250 4200 4250
-Wire Wire Line
-	3450 4150 4000 4150
-Wire Wire Line
-	3450 4250 3750 4250
+P 3900 4100
+F 0 "R13" H 3959 4146 50  0000 L CNN
+F 1 "4k7" H 3959 4055 50  0000 L CNN
+F 2 "Resistor_SMD:R_0603_1608Metric_Pad1.05x0.95mm_HandSolder" H 3900 4100 50  0001 C CNN
+F 3 "~" H 3900 4100 50  0001 C CNN
+	1    3900 4100
+	1    0    0    -1
+$EndComp
+Wire Wire Line
+	3900 4200 3900 4350
+Connection ~ 3900 4350
+Wire Wire Line
+	3900 4350 4350 4350
 NoConn ~ 3450 1750
 NoConn ~ 3450 1850
@@
 NoConn ~ 1650 3450
 NoConn ~ 1650 3550
-NoConn ~ 1650 3950
-NoConn ~ 1650 4050
-NoConn ~ 1650 4150
-NoConn ~ 1650 4250
-NoConn ~ 1650 4350
+NoConn ~ 3450 2950
+NoConn ~ 1650 4550
+NoConn ~ 1650 3750
+NoConn ~ 1650 4950
 NoConn ~ 1650 4450
-NoConn ~ 1650 4650
-NoConn ~ 1650 4750
 NoConn ~ 1650 4850
 NoConn ~ 3450 3850
-NoConn ~ 3450 3950
 NoConn ~ 3450 4050
-NoConn ~ 3450 4350
 NoConn ~ 3450 4450
 NoConn ~ 3450 4550
 NoConn ~ 3450 4650
 NoConn ~ 3450 4950
-NoConn ~ 3450 5350
 NoConn ~ 3450 5450
 NoConn ~ 3450 5750
@@
 Wire Wire Line
 	3750 3750 3450 3750
-Text Label 3750 5150 2    50   ~ 0
+Text Label 3750 3950 2    50   ~ 0
 LED1
-Text Label 3750 5250 2    50   ~ 0
+Text Label 3750 4150 2    50   ~ 0
 LED2
 Wire Wire Line
-	3750 5150 3450 5150
-Wire Wire Line
-	3750 5250 3450 5250
+	3750 3950 3450 3950
+Wire Wire Line
+	3750 4150 3450 4150
 $Comp
 L Device:R R?
@@
 Wire Wire Line
 	5750 5750 5850 5750
+Wire Wire Line
+	2350 1200 2350 1400
+Text HLabel 1650 4150 0    50   Input ~ 0
+PWR_VALID
+Text HLabel 1650 4250 0    50   Input ~ 0
+PWR_WARN
+Text HLabel 1650 4350 0    50   Input ~ 0
+PWR_CRITICAL
+$Comp
+L MCU_ST_STM32F4:STM32F407VGTx U3
+U 1 1 5FCFB0B5
+P 2550 4150
+F 0 "U3" H 2900 1500 50  0000 C CNN
+F 1 "STM32F407VGTx" H 3150 1400 50  0000 C CNN
+F 2 "Package_QFP:LQFP-100_14x14mm_P0.5mm" H 1850 1550 50  0001 R CNN
+F 3 "http://www.st.com/st-web-ui/static/active/en/resource/technical/document/datasheet/DM00037051.pdf" H 2550 4150 50  0001 C CNN
+	1    2550 4150
+	1    0    0    -1
+$EndComp
+Connection ~ 4150 4000
+Wire Wire Line
+	3450 4250 4150 4250
+Wire Wire Line
+	3450 4350 3900 4350
+NoConn ~ 3450 3550
+NoConn ~ 3450 3650
+NoConn ~ 3450 5150
+NoConn ~ 3450 5250
+NoConn ~ 3450 3450
+NoConn ~ 3450 2850
 $EndSCHEMATC
