File: KiCad/perpherals.sch (KiCad schematic (older format))
At the start: 15 parts

Commit message: Finalized schematic and created S/F associations
Parts:
- removed R? (x2): 4k7, symbol Device:R
- removed R?: 10k, symbol Device:R
- removed U?: RA-02_LORA, MODULE_RA-02_LORA, symbol Ra-02:RA-02_LORA
- added H1, H2, H3, H4: MountingHole, MountingHole:MountingHole_2.7mm_M2.5, symbol Mechanical:MountingHole
- added J5: RF_DATA, Connector_PinHeader_1.27mm:PinHeader_2x08_P1.27mm_Vertical_SMD, symbol Connector_Generic:Conn_02x08_Odd_Even
- added J6, J7, J8: GND, Connector_PinHeader_2.54mm:PinHeader_1x02_P2.54mm_Vertical, symbol Connector:Conn_01x02_Male
- added J9: COMM_ANT, Connector_Coaxial:SMA_Wurth_60312002114503_Vertical, symbol Connector:Conn_Coaxial
- added JP1: SCL, Jumper:SolderJumper-2_P1.3mm_Open_TrianglePad1.0x1.5mm, symbol Jumper:SolderJumper_2_Open
- added JP2: SDA, Jumper:SolderJumper-2_P1.3mm_Open_TrianglePad1.0x1.5mm, symbol Jumper:SolderJumper_2_Open
- added R1, R2, R4, R5: 22, Resistor_SMD:R_0603_1608Metric_Pad1.05x0.95mm_HandSolder, symbol Device:R_Small
- added R3: 10k, Resistor_SMD:R_0603_1608Metric_Pad1.05x0.95mm_HandSolder, symbol Device:R_Small
- added R6, R8: 4k7, Resistor_SMD:R_0603_1608Metric_Pad1.05x0.95mm_HandSolder, symbol Device:R_Small
- added U1: Ai-Thinker-Ra-01, RF_Module:Ai-Thinker-Ra-01-LoRa, symbol RF_Module:Ai-Thinker-Ra-01
- C1: renamed from C?; value 100n -> 1u; footprint (none) -> Capacitor_SMD:C_0603_1608Metric_Pad1.05x0.95mm_HandSolder
- F1: renamed from F?; footprint (none) -> Fuse:Fuse_0603_1608Metric_Pad1.05x0.95mm_HandSolder
- J1: renamed from J?; footprint (none) -> Connector_JST:JST_SHL_SM06B-SHLS-TF_1x06-1MP_P1.00mm_Horizontal
- J10: renamed from J?; footprint (none) -> Connector_PinHeader_2.54mm:PinHeader_1x03_P2.54mm_Horizontal
- J2: renamed from J?; footprint (none) -> Connector_JST:JST_SH_BM02B-SRSS-TB_1x02-1MP_P1.00mm_Vertical
- J3: renamed from J?; footprint (none) -> Connector_JST:JST_SH_BM03B-SRSS-TB_1x03-1MP_P1.00mm_Vertical
- J4: renamed from J?; footprint (none) -> Connector_JST:JST_SHL_SM05B-SHLS-TF_1x05-1MP_P1.00mm_Horizontal
- R10, R7, R9: renamed from R?; footprint (none) -> Resistor_SMD:R_0603_1608Metric_Pad1.05x0.95mm_HandSolder
- U2: renamed from U?; footprint SOP65P490X110-8N -> Libs:SOP65P490X110-8N
Connections:
- net labels added: CLK, GPIO_0, GPIO_1, GPIO_2, GPIO_3, MISO, MOSI, RF_ANT, VBAT
- wire segments 44 -> 61
- no-connect marks 0 -> 5
Other:
- note added: "RF board mechanical/GND connectors"
- note added: "optional compass i2c bus"
- note removed: "modify part and add sma antenna\n"
- moved on the sheet: C1, F1, J1, J10, J2, J3, J4, R10, R7, R9, U2

Commit message: Done some stuff
Parts:
- J9: footprint Connector_Coaxial:SMA_Wurth_60312002114503_Vertical -> Connector_Coaxial:U.FL_Molex_MCRF_73412-0110_Vertical
Changed lines of the file:
@@
 F 0 "J9" H 6850 3075 50  0000 L CNN
 F 1 "COMM_ANT" H 6850 2984 50  0000 L CNN
-F 2 "Connector_Coaxial:SMA_Wurth_60312002114503_Vertical" H 6750 3100 50  0001 C CNN
+F 2 "Connector_Coaxial:U.FL_Molex_MCRF_73412-0110_Vertical" H 6750 3100 50  0001 C CNN
 F 3 " ~" H 6750 3100 50  0001 C CNN
 	1    6750 3100

Commit message: Semi-final flight computer version
Parts:
- removed H1, H2, H3, H4: MountingHole, MountingHole:MountingHole_2.7mm_M2.5, symbol Mechanical:MountingHole
- removed J8: GND, Connector_PinHeader_2.54mm:PinHeader_1x02_P2.54mm_Vertical, symbol Connector:Conn_01x02_Male
- added H1, H2, H3, H4: MountingHole_Pad, MountingHole:MountingHole_2.7mm_M2.5_Pad_Via, symbol Mechanical:MountingHole_Pad
Connections:
- net GND: now also H1.1, H2.1, H3.1, H4.1
- net SCL: now also JP1.2 (B); no longer JP2.2 (B)
- net SDA: now also JP2.2 (B); no longer JP1.2 (B)
Changed lines of the file:
@@
 	0    1    1    0
 $EndComp
-Text HLabel 2250 3200 3    50   Input ~ 0
+Text HLabel 1950 3200 3    50   Input ~ 0
 SCL
-Text HLabel 1950 3200 3    50   BiDi ~ 0
+Text HLabel 2250 3200 3    50   BiDi ~ 0
 SDA
 Text Notes 1700 3500 0    50   ~ 0
@@
 	6350 1650 6350 1600
 Connection ~ 6350 1600
-$Comp
-L Connector:Conn_01x02_Male J8
-U 1 1 60189EFB
-P 6500 1500
-F 0 "J8" H 6608 1681 50  0000 C CNN
-F 1 "GND" H 6608 1590 50  0000 C CNN
-F 2 "Connector_PinHeader_2.54mm:PinHeader_1x02_P2.54mm_Vertical" H 6500 1500 50  0001 C CNN
-F 3 "~" H 6500 1500 50  0001 C CNN
-	1    6500 1500
-	1    0    0    -1
-$EndComp
-Wire Wire Line
-	6700 1500 6750 1500
-Wire Wire Line
-	6750 1500 6750 1600
-Wire Wire Line
-	6750 1600 6700 1600
+Text Notes 5350 1250 0    50   ~ 0
+RF board mechanical/GND connectors
+$Comp
+L Mechanical:MountingHole_Pad H1
+U 1 1 5FE37D1F
+P 2100 6850
+F 0 "H1" H 2200 6899 50  0000 L CNN
+F 1 "MountingHole_Pad" H 2200 6808 50  0000 L CNN
+F 2 "MountingHole:MountingHole_2.7mm_M2.5_Pad_Via" H 2100 6850 50  0001 C CNN
+F 3 "~" H 2100 6850 50  0001 C CNN
+	1    2100 6850
+	1    0    0    -1
+$EndComp
+$Comp
+L Mechanical:MountingHole_Pad H2
+U 1 1 5FE3856E
+P 3050 6850
+F 0 "H2" H 3150 6899 50  0000 L CNN
+F 1 "MountingHole_Pad" H 3150 6808 50  0000 L CNN
+F 2 "MountingHole:MountingHole_2.7mm_M2.5_Pad_Via" H 3050 6850 50  0001 C CNN
+F 3 "~" H 3050 6850 50  0001 C CNN
+	1    3050 6850
+	1    0    0    -1
+$EndComp
+$Comp
+L Mechanical:MountingHole_Pad H3
+U 1 1 5FE397C2
+P 4000 6850
+F 0 "H3" H 4100 6899 50  0000 L CNN
+F 1 "MountingHole_Pad" H 4100 6808 50  0000 L CNN
+F 2 "MountingHole:MountingHole_2.7mm_M2.5_Pad_Via" H 4000 6850 50  0001 C CNN
+F 3 "~" H 4000 6850 50  0001 C CNN
+	1    4000 6850
+	1    0    0    -1
+$EndComp
+$Comp
+L Mechanical:MountingHole_Pad H4
+U 1 1 5FE3A96E
+P 4950 6850
+F 0 "H4" H 5050 6899 50  0000 L CNN
+F 1 "MountingHole_Pad" H 5050 6808 50  0000 L CNN
+F 2 "MountingHole:MountingHole_2.7mm_M2.5_Pad_Via" H 4950 6850 50  0001 C CNN
+F 3 "~" H 4950 6850 50  0001 C CNN
+	1    4950 6850
+	1    0    0    -1
+$EndComp
 $Comp
 L power:GND #PWR0120
-U 1 1 60189F04
-P 6750 1650
-F 0 "#PWR0120" H 6750 1400 50  0001 C CNN
-F 1 "GND" H 6755 1477 50  0000 C CNN
-F 2 "" H 6750 1650 50  0001 C CNN
-F 3 "" H 6750 1650 50  0001 C CNN
-	1    6750 1650
-	1    0    0    -1
-$EndComp
-Wire Wire Line
-	6750 1650 6750 1600
-Connection ~ 6750 1600
-Text Notes 5550 1250 0    50   ~ 0
-RF board mechanical/GND connectors
-$Comp
-L Mechanical:MountingHole H1
-U 1 1 602102E8
-P 2100 7000
-F 0 "H1" H 2200 7046 50  0000 L CNN
-F 1 "MountingHole" H 2200 6955 50  0000 L CNN
-F 2 "MountingHole:MountingHole_2.7mm_M2.5" H 2100 7000 50  0001 C CNN
-F 3 "~" H 2100 7000 50  0001 C CNN
-	1    2100 7000
-	1    0    0    -1
-$EndComp
-$Comp
-L Mechanical:MountingHole H2
-U 1 1 602113EA
-P 3050 7000
-F 0 "H2" H 3150 7046 50  0000 L CNN
-F 1 "MountingHole" H 3150 6955 50  0000 L CNN
-F 2 "MountingHole:MountingHole_2.7mm_M2.5" H 3050 7000 50  0001 C CNN
-F 3 "~" H 3050 7000 50  0001 C CNN
-	1    3050 7000
-	1    0    0    -1
-$EndComp
-$Comp
-L Mechanical:MountingHole H3
-U 1 1 602191CF
-P 4000 7000
-F 0 "H3" H 4100 7046 50  0000 L CNN
-F 1 "MountingHole" H 4100 6955 50  0000 L CNN
-F 2 "MountingHole:MountingHole_2.7mm_M2.5" H 4000 7000 50  0001 C CNN
-F 3 "~" H 4000 7000 50  0001 C CNN
-	1    4000 7000
-	1    0    0    -1
-$EndComp
-$Comp
-L Mechanical:MountingHole H4
-U 1 1 602191D5
-P 4950 7000
-F 0 "H4" H 5050 7046 50  0000 L CNN
-F 1 "MountingHole" H 5050 6955 50  0000 L CNN
-F 2 "MountingHole:MountingHole_2.7mm_M2.5" H 4950 7000 50  0001 C CNN
-F 3 "~" H 4950 7000 50  0001 C CNN
-	1    4950 7000
-	1    0    0    -1
-$EndComp
+U 1 1 5FE3E34B
+P 2100 6950
+F 0 "#PWR0120" H 2100 6700 50  0001 C CNN
+F 1 "GND" H 2105 6777 50  0000 C CNN
+F 2 "" H 2100 6950 50  0001 C CNN
+F 3 "" H 2100 6950 50  0001 C CNN
+	1    2100 6950
+	1    0    0    -1
+$EndComp
+$Comp
+L power:GND #PWR0122
+U 1 1 5FE3EBD3
+P 3050 6950
+F 0 "#PWR0122" H 3050 6700 50  0001 C CNN
+F 1 "GND" H 3055 6777 50  0000 C CNN
+F 2 "" H 3050 6950 50  0001 C CNN
+F 3 "" H 3050 6950 50  0001 C CNN
+	1    3050 6950
+	1    0    0    -1
+$EndComp
+$Comp
+L power:GND #PWR0123
+U 1 1 5FE3F02C
+P 4000 6950
+F 0 "#PWR0123" H 4000 6700 50  0001 C CNN
+F 1 "GND" H 4005 6777 50  0000 C CNN
+F 2 "" H 4000 6950 50  0001 C CNN
+F 3 "" H 4000 6950 50  0001 C CNN
+	1    4000 6950
+	1    0    0    -1
+$EndComp
+$Comp
+L power:GND #PWR0124
+U 1 1 5FE3F49B
+P 4950 6950
+F 0 "#PWR0124" H 4950 6700 50  0001 C CNN
+F 1 "GND" H 4955 6777 50  0000 C CNN
+F 2 "" H 4950 6950 50  0001 C CNN
+F 3 "" H 4950 6950 50  0001 C CNN
+	1    4950 6950
+	1    0    0    -1
+$EndComp
