File: KiCad/rpi_cm4.sch (KiCad schematic (older format))
At the start: 14 parts, among them J15 DF40C-100DS-0.4V(51), J16 DF40C-100DS-0.4V(51), J17 RPI_GPIO, P1 USB_SDR, U4 SN74LVC1G125DCKT, U5 USBLC6-2SC6, U6 SN74LVC1G125DCKT

Commit message: Dirty production PCBs commit
Connections:
- net GPIO_5: now also J17.5 (Pin_5); no longer J17.6 (Pin_6)
- net GPIO_4: now reaches J15.54
- net GPIO_4: now also J17.6 (Pin_6)
- net GPIO_6: no longer names the net of J15.30
- net GPIO_6: no longer J17.5 (Pin_5)
Changed lines of the file:
@@
 	2450 2400 2150 2400
 Wire Wire Line
-	2450 2500 2150 2500
+	2450 3700 2150 3700
 Wire Wire Line
 	2450 2700 2150 2700
@@
 Text Label 2450 2400 2    50   ~ 0
 GPIO_13
-Text Label 2450 2500 2    50   ~ 0
-GPIO_6
+Text Label 2450 3700 2    50   ~ 0
+GPIO_4
 Text Label 2450 2700 2    50   ~ 0
 GPIO_5
@@
 NoConn ~ 2150 3400
 NoConn ~ 2150 3500
-NoConn ~ 2150 3700
 NoConn ~ 2150 3800
 NoConn ~ 2150 3900
@@
 $EndComp
 Text Label 8850 5050 0    50   ~ 0
-GPIO_5
+GPIO_4
 Wire Wire Line
 	8850 5050 9200 5050
@@
 	8850 5150 9200 5150
 Text Label 8850 5150 0    50   ~ 0
-GPIO_6
+GPIO_5
 Wire Wire Line
 	8850 5250 9200 5250
@@
 	1    0    0    -1
 $EndComp
+NoConn ~ 2150 2500
 $EndSCHEMATC
